Commit message: 関節制限/

File: ur_moveit_config/srdf/ur_macro.srdf.xacro (robot description, xacro)
@@ -12,5 +12,6 @@
     <!--SUBGROUPS - Groups can also be formed by referencing to already defined group names-->
     <group name="${prefix}${name}_manipulator">
-      <chain base_link="${prefix}base_link" tip_link="${prefix}tool0" />
+      <!-- <chain base_link="${prefix}base_link" tip_link="${prefix}tool0" /> -->
+      <chain base_link="${prefix}base_link" tip_link="endeffector_cutter" />
     </group>
     <!--GROUP STATES - Purpose - Define a named state for a particular group, in terms of joint values. This is useful to define states like 'folded arms'-->
@@ -39,4 +40,20 @@
       <joint name="${prefix}wrist_3_joint" value="-0.11" />
     </group_state>
+    <group_state name="${prefix}servo_set" group="${prefix}${name}_manipulator">
+      <joint name="${prefix}elbow_joint" value="2.24146" />
+      <joint name="${prefix}shoulder_lift_joint" value="-1.6054" />
+      <joint name="${prefix}shoulder_pan_joint" value="1.634" />
+      <joint name="${prefix}wrist_1_joint" value="-0.6578" />
+      <joint name="${prefix}wrist_2_joint" value="1.64835" />
+      <joint name="${prefix}wrist_3_joint" value="-0.028" /> <!-- -0.028 -->
+    </group_state>
+    <group_state name="${prefix}harvest_set" group="${prefix}${name}_manipulator">
+      <joint name="${prefix}elbow_joint" value="2.2096994558917444" />
+      <joint name="${prefix}shoulder_lift_joint" value="-2.0010177097716273" />
+      <joint name="${prefix}shoulder_pan_joint" value="2.2522974014282227" />
+      <joint name="${prefix}wrist_1_joint" value="-0.2257133287242432" />
+      <joint name="${prefix}wrist_2_joint" value="2.2583630084991455" />
+      <joint name="${prefix}wrist_3_joint" value="-0.008907143269674123" />
+    </group_state>
     <!--END EFFECTOR - Purpose - Represent information about an end effector.-->
     <!--VIRTUAL JOINT - Purpose - this element defines a virtual joint between a robot link and an external frame of reference (considered fixed with respect to the robot)-->
@@ -53,4 +70,6 @@
     <disable_collisions link1="${prefix}wrist_1_link" link2="${prefix}wrist_3_link" reason="Never" />
     <disable_collisions link1="${prefix}wrist_2_link" link2="${prefix}wrist_3_link" reason="Adjacent" />
+    <disable_collisions link1="${prefix}tool0" link2="endeffector_type5" reason="Adjacent" />
+    <disable_collisions link1="endeffector_type5" link2="endeffector_cutter" reason="Adjacent" />
   </xacro:macro>
 </robot>

Commit message: 模型収穫250725

File: ur_moveit_config/srdf/ur_macro.srdf.xacro (robot description, xacro)
@@ -49,10 +49,18 @@
     </group_state>
     <group_state name="${prefix}harvest_set" group="${prefix}${name}_manipulator">
-      <joint name="${prefix}elbow_joint" value="2.2096994558917444" />
-      <joint name="${prefix}shoulder_lift_joint" value="-2.0010177097716273" />
-      <joint name="${prefix}shoulder_pan_joint" value="2.2522974014282227" />
-      <joint name="${prefix}wrist_1_joint" value="-0.2257133287242432" />
-      <joint name="${prefix}wrist_2_joint" value="2.2583630084991455" />
-      <joint name="${prefix}wrist_3_joint" value="-0.008907143269674123" />
+      <joint name="${prefix}elbow_joint" value="2.187139381739011" />
+      <joint name="${prefix}shoulder_lift_joint" value="-2.043222502923897" />
+      <joint name="${prefix}shoulder_pan_joint" value="1.6987447853438469" />
+      <joint name="${prefix}wrist_1_joint" value="-0.16578364100649842" />
+      <joint name="${prefix}wrist_2_joint" value="1.7132108772666321" />
+      <joint name="${prefix}wrist_3_joint" value="-0.029275631321143938" />
+    </group_state>
+    <group_state name="${prefix}new_harvest_set" group="${prefix}${name}_manipulator">
+      <joint name="${prefix}elbow_joint" value="2.4783" />
+      <joint name="${prefix}shoulder_lift_joint" value="-1.8675" />
+      <joint name="${prefix}shoulder_pan_joint" value="1.6929" />
+      <joint name="${prefix}wrist_1_joint" value="-3.7873" />
+      <joint name="${prefix}wrist_2_joint" value="-1.6929" />
+      <joint name="${prefix}wrist_3_joint" value="3.1415" />
     </group_state>
     <!--END EFFECTOR - Purpose - Represent information about an end effector.-->
@@ -70,5 +78,8 @@
     <disable_collisions link1="${prefix}wrist_1_link" link2="${prefix}wrist_3_link" reason="Never" />
     <disable_collisions link1="${prefix}wrist_2_link" link2="${prefix}wrist_3_link" reason="Adjacent" />
-    <disable_collisions link1="${prefix}tool0" link2="endeffector_type5" reason="Adjacent" />
+    <disable_collisions link1="${prefix}tool0" link2="endeffector_base" reason="Adjacent" />
+    <disable_collisions link1="endeffector_base" link2="head_camera_link" reason="Adjacent" />
+    <disable_collisions link1="endeffector_base" link2="endeffector_type5" reason="Adjacent" />
+    <disable_collisions link1="head_camera_link" link2="realsense_cable" reason="Adjacent" />
     <disable_collisions link1="endeffector_type5" link2="endeffector_cutter" reason="Adjacent" />
   </xacro:macro>

Commit message: 姿勢を削除

File: ur_moveit_config/srdf/ur_macro.srdf.xacro (robot description, xacro)
@@ -48,12 +48,4 @@
       <joint name="${prefix}wrist_3_joint" value="-0.028" /> <!-- -0.028 -->
     </group_state>
-    <group_state name="${prefix}harvest_set" group="${prefix}${name}_manipulator">
-      <joint name="${prefix}elbow_joint" value="2.187139381739011" />
-      <joint name="${prefix}shoulder_lift_joint" value="-2.043222502923897" />
-      <joint name="${prefix}shoulder_pan_joint" value="1.6987447853438469" />
-      <joint name="${prefix}wrist_1_joint" value="-0.16578364100649842" />
-      <joint name="${prefix}wrist_2_joint" value="1.7132108772666321" />
-      <joint name="${prefix}wrist_3_joint" value="-0.029275631321143938" />
-    </group_state>
     <group_state name="${prefix}new_harvest_set" group="${prefix}${name}_manipulator">
       <joint name="${prefix}elbow_joint" value="2.4783" />
@@ -64,4 +56,12 @@
       <joint name="${prefix}wrist_3_joint" value="3.1415" />
     </group_state>
+    <!-- <group_state name="${prefix}new_harvest_set" group="${prefix}${name}_manipulator">
+      <joint name="${prefix}elbow_joint" value="2.616568152104513" />
+      <joint name="${prefix}shoulder_lift_joint" value="-2.2550112209715785" />
+      <joint name="${prefix}shoulder_pan_joint" value="2.244324207305908" />
+      <joint name="${prefix}wrist_1_joint" value="-3.505115648309225" />
+      <joint name="${prefix}wrist_2_joint" value="-2.244192425404684" />
+      <joint name="${prefix}wrist_3_joint" value="3.144463300704956" />
+    </group_state> -->
     <!--END EFFECTOR - Purpose - Represent information about an end effector.-->
     <!--VIRTUAL JOINT - Purpose - this element defines a virtual joint between a robot link and an external frame of reference (considered fixed with respect to the robot)-->

Commit message: change collision flag

File: ur_moveit_config/srdf/ur_macro.srdf.xacro (robot description, xacro)
@@ -48,5 +48,5 @@
       <joint name="${prefix}wrist_3_joint" value="-0.028" /> <!-- -0.028 -->
     </group_state>
-    <group_state name="${prefix}new_harvest_set" group="${prefix}${name}_manipulator">
+    <!-- <group_state name="${prefix}new_harvest_set" group="${prefix}${name}_manipulator">
       <joint name="${prefix}elbow_joint" value="2.4783" />
       <joint name="${prefix}shoulder_lift_joint" value="-1.8675" />
@@ -55,13 +55,13 @@
       <joint name="${prefix}wrist_2_joint" value="-1.6929" />
       <joint name="${prefix}wrist_3_joint" value="3.1415" />
+    </group_state> -->
+    <group_state name="${prefix}new_harvest_set" group="${prefix}${name}_manipulator">
+      <joint name="${prefix}elbow_joint" value="2.2812183539019983" />
+      <joint name="${prefix}shoulder_lift_joint" value="-1.6140600643553675" />
+      <joint name="${prefix}shoulder_pan_joint" value="0.16587185859680176" />
+      <joint name="${prefix}wrist_1_joint" value="-4.0158709488310755" />
+      <joint name="${prefix}wrist_2_joint" value="-0.16943198839296514" />
+      <joint name="${prefix}wrist_3_joint" value="3.34975004196167" />
     </group_state>
-    <!-- <group_state name="${prefix}new_harvest_set" group="${prefix}${name}_manipulator">
-      <joint name="${prefix}elbow_joint" value="2.616568152104513" />
-      <joint name="${prefix}shoulder_lift_joint" value="-2.2550112209715785" />
-      <joint name="${prefix}shoulder_pan_joint" value="2.244324207305908" />
-      <joint name="${prefix}wrist_1_joint" value="-3.505115648309225" />
-      <joint name="${prefix}wrist_2_joint" value="-2.244192425404684" />
-      <joint name="${prefix}wrist_3_joint" value="3.144463300704956" />
-    </group_state> -->
     <!--END EFFECTOR - Purpose - Represent information about an end effector.-->
     <!--VIRTUAL JOINT - Purpose - this element defines a virtual joint between a robot link and an external frame of reference (considered fixed with respect to the robot)-->

Commit message: add_vertical_arm_pose

File: ur_moveit_config/srdf/ur_macro.srdf.xacro (robot description, xacro)
@@ -64,4 +64,12 @@
       <joint name="${prefix}wrist_3_joint" value="3.34975004196167" />
     </group_state>
+    <group_state name="${prefix}vertical_harvest_set" group="${prefix}${name}_manipulator">
+      <joint name="${prefix}elbow_joint" value="2.44346" />
+      <joint name="${prefix}shoulder_lift_joint" value="-1.65806" />
+      <joint name="${prefix}shoulder_pan_joint" value="0.0" />
+      <joint name="${prefix}wrist_1_joint" value="-2.35619" />
+      <joint name="${prefix}wrist_2_joint" value="-1.5708" />
+      <joint name="${prefix}wrist_3_joint" value="-1.5708" />
+    </group_state>
     <!--END EFFECTOR - Purpose - Represent information about an end effector.-->
     <!--VIRTUAL JOINT - Purpose - this element defines a virtual joint between a robot link and an external frame of reference (considered fixed with respect to the robot)-->

Commit message: add vertical_harvest_set_wide

File: ur_moveit_config/srdf/ur_macro.srdf.xacro (robot description, xacro)
@@ -72,4 +72,12 @@
       <joint name="${prefix}wrist_3_joint" value="-1.5708" />
     </group_state>
+    <group_state name="${prefix}vertical_harvest_set_wide" group="${prefix}${name}_manipulator">
+      <joint name="${prefix}elbow_joint" value="2.14675" />
+      <joint name="${prefix}shoulder_lift_joint" value="-1.37881" />
+      <joint name="${prefix}shoulder_pan_joint" value="0.0" />
+      <joint name="${prefix}wrist_1_joint" value="-2.33874" />
+      <joint name="${prefix}wrist_2_joint" value="-1.5708" />
+      <joint name="${prefix}wrist_3_joint" value="-1.5708" />
+    </group_state>
     <!--END EFFECTOR - Purpose - Represent information about an end effector.-->
     <!--VIRTUAL JOINT - Purpose - this element defines a virtual joint between a robot link and an external frame of reference (considered fixed with respect to the robot)-->
